Commit message: Added Sensor Functionality

File: limo_description/urdf/limo_xacro.xacro (robot description, xacro)
@@ -15,15 +15,15 @@
             </visual>
             <collision>
-              <origin xyz="0 ${wheel_length/2} 0" rpy="1.57 0 0" />
-              <geometry>
-                  <cylinder length="${wheel_length}" radius="${wheel_radius}" />
-              </geometry>
+                <origin xyz="0 ${wheel_length/2} 0" rpy="1.57 0 0" />
+                <geometry>
+                    <cylinder length="${wheel_length}" radius="${wheel_radius}" />
+                </geometry>
             </collision>
         </link>
         <joint name="${wheel_prefix}_wheel" type="continuous">
-            <parent link="${parent_prefix}"/>
-            <child link="${wheel_prefix}_wheel_link"/>
-            <xacro:insert_block name="joint_pose"/>
-            <axis xyz="0 ${reflect*1} 0"/>
+            <parent link="${parent_prefix}" />
+            <child link="${wheel_prefix}_wheel_link" />
+            <xacro:insert_block name="joint_pose" />
+            <axis xyz="0 ${reflect*1} 0" />
         </joint>
     </xacro:macro>
@@ -32,6 +32,6 @@
             <pose>0 0 0 0 0 0</pose>
             <inertial>
-                <mass value="0.1"/>
-                <origin xyz="0.0 0 0" rpy="0 0 0"/>
+                <mass value="0.1" />
+                <origin xyz="0.0 0 0" rpy="0 0 0" />
                 <inertia
                     ixx="1e-6" ixy="0" ixz="0"
@@ -41,7 +41,7 @@
             </inertial>
             <visual name='laser_visual'>
-                <origin xyz="0 0 0" rpy="0 0 0"/>
-                <geometry>
-                    <cylinder radius="0.02" length="0.01"/>
+                <origin xyz="0 0 0" rpy="0 0 0" />
+                <geometry>
+                    <cylinder radius="0.02" length="0.01" />
                 </geometry>
                 <material name='laser_material'>
@@ -53,17 +53,46 @@
             </visual>
             <collision name='laser_collision'>
-                <origin xyz="0 0 0" rpy="0 0 0"/>
-                <geometry>
-                    <cylinder radius="0.032" length="0.016"/>
+                <origin xyz="0 0 0" rpy="0 0 0" />
+                <geometry>
+                    <cylinder radius="0.032" length="0.016" />
                 </geometry>
             </collision>
         </link>
         <joint type="fixed" name="laser_joint">
-            <xacro:insert_block name="joint_pose"/>
-            <child link="${frame_prefix}_link"/>
-            <parent link="${parent_prefix}"/>
+            <xacro:insert_block name="joint_pose" />
+            <child link="${frame_prefix}_link" />
+            <parent link="${parent_prefix}" />
         </joint>
         <gazebo reference="${frame_prefix}_link">
             <material>Gazebo/Yellow</material>
+            <sensor name="laser" type="ray" update_rate="10">
+                <visualize>false</visualize>
+                <ray>
+                    <scan>
+                        <horizontal>
+                            <samples>360</samples>
+                            <resolution>1</resolution>
+                            <min_angle>-3.14</min_angle>
+                            <max_angle>3.14</max_angle>
+                        </horizontal>
+                    </scan>
+                    <range>
+                        <min>0.3</min>
+                        <max>12</max>
+                        <resolution>0.01</resolution>
+                    </range>
+                </ray>
+                <plugin name="laser_controller" filename="libgazebo_ros_ray_sensor.so">
+                    <ros>
+                        <argument>~/out:=scan</argument>
+                    </ros>
+                    <output_type>sensor_msg/LaserScan</output_type>
+                    <frame_name>${frame_prefix}_link</frame_name>
+                </plugin>
+                <parent link="parent_link" />
+                <origin xyz="0.0 0.0 0.0" rpy="0.0 0.0 0.0" />
+                <!-- Sensor
+                |camera,ray,imu,magnetometer,gps,force_torque,contact,sonar,rfidtag,rfid| -->
+            </sensor>
         </gazebo>
     </xacro:macro>
@@ -72,6 +101,6 @@
             <pose>0 0 0 0 0 0</pose>
             <inertial>
-                <mass value="0.1"/>
-                <origin xyz="0.0 0 0" rpy="0 0 0"/>
+                <mass value="0.1" />
+                <origin xyz="0.0 0 0" rpy="0 0 0" />
                 <inertia
                     ixx="1e-6" ixy="0" ixz="0"
@@ -81,7 +110,7 @@
             </inertial>
             <visual name='depth_camera_visual'>
-                <origin xyz="0 0 0" rpy="0 0 0"/>
-                <geometry>
-                    <box size="0.02 0.06 0.015"/>
+                <origin xyz="0 0 0" rpy="0 0 0" />
+                <geometry>
+                    <box size="0.02 0.06 0.015" />
                 </geometry>
                 <material name='depth_camera_material'>
@@ -93,23 +122,37 @@
             </visual>
             <collision name='depth_camera_collision'>
-                <origin xyz="0 0 0" rpy="0 0 0"/>
-                <geometry>
-                    <box size="0.02 0.06 0.015"/>
+                <origin xyz="0 0 0" rpy="0 0 0" />
+                <geometry>
+                    <box size="0.02 0.06 0.015" />
                 </geometry>
             </collision>
         </link>
         <joint type="fixed" name="depth_camera_joint">
-            <xacro:insert_block name="joint_pose"/>
-            <child link="${frame_prefix}_link"/>
-            <parent link="${parent_prefix}"/>
+            <xacro:insert_block name="joint_pose" />
+            <child link="${frame_prefix}_link" />
+            <parent link="${parent_prefix}" />
         </joint>
         <link name="depth_link"></link>
         <joint name="${frame_prefix}_to_camera_joint" type="fixed">
-            <origin xyz="0 0 0" rpy="${-M_PI/2} 0 ${-M_PI/2} "/>
-            <parent link="${frame_prefix}_link"/>
-            <child link="depth_link"/>
-          </joint>
+            <origin xyz="0 0 0" rpy="${-M_PI/2} 0 ${-M_PI/2} " />
+            <parent link="${frame_prefix}_link" />
+            <child link="depth_link" />
+        </joint>
         <gazebo reference="${frame_prefix}_link">
             <material>Gazebo/Yellow</material>
+            <sensor name="depth_camera" type="depth" update_rate="10">
+                <visualize>true</visualize>
+                <camera>
+                    <image width="640" height="480" hfov="1.5708" format="B8R8G8" near="0.05"
+                        far="8.0" />
+                </camera>
+                <plugin name="camera_controller" filename="libgazebo_ros_camera.so">
+                    <frame_name>depth_link</frame_name>
+                    <min_depth>0.1</min_depth>
+                    <max_depth>100</max_depth>
+                </plugin>
+                <parent link="parent_link" />
+                <origin xyz="0.0 0.0 0.0" rpy="0.0 0.0 0.0" />
+            </sensor>
         </gazebo>
     </xacro:macro>
@@ -118,6 +161,6 @@
             <pose>0 0 0 0 0 0</pose>
             <inertial>
-                <mass value="0.01"/>
-                <origin xyz="0.0 0 0" rpy="0 0 0"/>
+                <mass value="0.01" />
+                <origin xyz="0.0 0 0" rpy="0 0 0" />
                 <inertia
                     ixx="1e-7" ixy="0" ixz="0"
@@ -127,7 +170,7 @@
             </inertial>
             <visual name='imu_visual'>
-                <origin xyz="0 0 0" rpy="0 0 0"/>
-                <geometry>
-                    <box size="0.001 0.001 0.001"/>
+                <origin xyz="0 0 0" rpy="0 0 0" />
+                <geometry>
+                    <box size="0.001 0.001 0.001" />
                 </geometry>
                 <material name='imu_material'>
@@ -139,17 +182,25 @@
             </visual>
             <collision name='imu_collision'>
-                <origin xyz="0 0 0" rpy="0 0 0"/>
-                <geometry>
-                    <box size="0.001 0.001 0.001"/>
+                <origin xyz="0 0 0" rpy="0 0 0" />
+                <geometry>
+                    <box size="0.001 0.001 0.001" />
                 </geometry>
             </collision>
         </link>
         <joint type="fixed" name="imu_joint">
-            <xacro:insert_block name="joint_pose"/>
-            <child link="${frame_prefix}_link"/>
-            <parent link="${parent_prefix}"/>
+            <xacro:insert_block name="joint_pose" />
+            <child link="${frame_prefix}_link" />
+            <parent link="${parent_prefix}" />
         </joint>
         <gazebo reference="${frame_prefix}_link">
             <material>Gazebo/Yellow</material>
+            <plugin name="imu_plugin" filename="libgazebo_ros_imu.so">
+                <alwaysOn>true</alwaysOn>
+                <bodyName>base_footprint</bodyName>
+                <topicName>imu</topicName>
+                <serviceName>imu_service</serviceName>
+                <gaussianNoise>0.0</gaussianNoise>
+                <updateRate>20.0</updateRate>
+            </plugin>
         </gazebo>
     </xacro:macro>
