Commit message: Added simulation table with: Trees, Working traffic light

File: limo_description/urdf/limo_four_diff.xacro (robot description, xacro)
@@ -26,5 +26,5 @@
             <origin xyz="0 0 -0.15" rpy="0 0 1.57" />
             <geometry>
-                <mesh filename="package://limo_description/meshes/limo_base.dae" scale="1 1 1"/>
+                <mesh filename="package://limo_description/meshes/limo_base_simple.dae" scale="1 1 1"/>
             </geometry>
         </visual>
